Commit message: feat: more accurate urdf with meshes

File: TeamCode/src/main/assets/robot.urdf (robot description, URDF)
Before this commit: robot decode_robot, 17 links, 16 joints
Links:
- link base_link: geometry collision box size=0.39557406 0.4367 0.1016; visual mesh filename=robotMeshes/robot frame.stl scale=0.001 0.001 0.001
- link bl_wheel: geometry collision cylinder length=0.05 radius=0.05; visual mesh filename=robotMeshes/wheel.stl scale=0.001 0.001 0.001
- link br_wheel: geometry collision cylinder length=0.05 radius=0.05; visual mesh filename=robotMeshes/wheel.stl scale=0.001 0.001 0.001
- link fl_wheel: geometry collision cylinder length=0.048 radius=0.048; visual mesh filename=robotMeshes/wheel.stl scale=0.001 0.001 0.001
- link fr_wheel: geometry collision cylinder length=0.048 radius=0.048; visual mesh filename=robotMeshes/wheel.stl scale=0.001 0.001 0.001
- link intake_link: geometry 
- link turret_link: geometry visual mesh filename=robotMeshes/shooter.stl scale=0.001 0.001 0.001
Joints:
- joint bl_wheel_joint: origin xyz=-0.15 0.15 0 rpy=-1.5708 0 0 -> xyz=-0.13278703 0.1538125 0.04 rpy=-1.57079632679 0 0
- joint br_wheel_joint: origin xyz=-0.15 -0.15 0 rpy=-1.5708 0 0 -> xyz=-0.13278703 -0.1538125 0.04 rpy=-1.57079632679 0 0
- joint fl_wheel_joint: origin xyz=0.15 0.15 0 rpy=-1.5708 0 0 -> xyz=0.13278703 0.1538125 0.04 rpy=-1.57079632679 0 0
- joint fr_wheel_joint: origin xyz=0.15 -0.15 0 rpy=-1.5708 0 0 -> xyz=0.13278703 -0.1538125 0.04 rpy=-1.57079632679 0 0
- joint intake_joint: origin xyz=0.25 0 0 rpy=0 1.5708 0 -> xyz=0.25 0 1 rpy=0 1.5708 0
- joint turret_joint: limit lower=-1.5708 upper=1.5708 effort=20 velocity=10 -> (none); origin xyz=0 0 0.15 rpy=0 0 0 -> xyz=-0.039962 0 0.22744 rpy=0 0 0; type revolute -> continuous

Commit message: feat: mpc change

File: TeamCode/src/main/assets/robot.urdf (robot description, URDF)
Before this commit: robot decode_robot, 17 links, 16 joints
Links:
- link base_link: mass 10.0 -> 15.0

Commit message: fix(drake): gamepad control + in progress game element interaction

File: TeamCode/src/main/assets/robot.urdf (robot description, URDF)
Before this commit: robot decode_robot, 17 links, 16 joints
Links:
- link turret_link: geometry visual mesh filename=robotMeshes/shooter.stl scale=1.0 1.0 1.0

Commit message: feat(drake): intake+shooting working

File: TeamCode/src/main/assets/robot.urdf (robot description, URDF)
Before this commit: robot decode_robot, 17 links, 16 joints
Links:
- removed link div1
- removed link div2
- removed link div3
- removed link hood_seg1
- removed link hood_seg2
- removed link hood_seg3
- link base_link: geometry collision box size=0.4367 0.39557406 0.1016; visual mesh filename=robotMeshes/robot frame.stl scale=0.001 0.001 0.001
- link intake_link: geometry visual cylinder length=0.2 radius=0.03
- link transfer_ramp: geometry visual box size=0.12 0.08 0.02
Joints:
- removed joint div1_joint
- removed joint div2_joint
- removed joint div3_joint
- removed joint h1
- removed joint h2
- removed joint h3
- joint intake_joint: origin xyz=0.25 0 1 rpy=0 1.5708 0 -> xyz=0.2 0 0.128 rpy=0 1.5708 1.5708
- joint turret_joint: origin xyz=-0.039962 0 0.22744 rpy=0 0 0 -> xyz=-0.039962 0 0.204265 rpy=0 0 0

Commit message: feat(drake): better intake simulation

File: TeamCode/src/main/assets/robot.urdf (robot description, URDF)
Before this commit: robot decode_robot, 11 links, 10 joints
Links:
- link intake_link: geometry collision cylinder length=0.3 radius=0.03; visual cylinder length=0.2 radius=0.03
Joints:
- joint intake_joint: origin xyz=0.2 0 0.128 rpy=0 1.5708 1.5708 -> xyz=0.2 0 0.1 rpy=0 1.5708 4.7124
